File: frosting.kicad_pcb (KiCad board)
At the start: 4 copper layers, 70 x 82.5 mm, 51 parts, among them J101 HRO-Type-C-31-M-12, J102 iCESugar-Pro, SW101 USER3, SW102 USER2, SW103 USER1, U101 SRV05-4, U102 XC6206

Commit message: clean erc drc
Parts:
- added D109: 5VOK, LED_SMD:LED_0603_1608Metric, F.Cu at (161.2, 70.1)
- added D110: 3V3OK, LED_SMD:LED_0603_1608Metric, F.Cu at (164.1, 70.1)
- added G***: LOGO, LOGO, F.Cu at (151.2, 102.7)
- added G***: LOGO, LOGO, B.Cu at (150.3, 101.8)
- added H101: M3, MountingHole:MountingHole_3.2mm_M3_DIN965_Pad, F.Cu at (178.9, 68.3)
- added H102: M3, MountingHole:MountingHole_3.2mm_M3_DIN965_Pad, F.Cu at (118.2, 68.3)
- added H103: M3, MountingHole:MountingHole_3.2mm_M3_DIN965_Pad, F.Cu at (148.3, 133.5)
- added R117: 5k1, Resistor_SMD:R_0402_1005Metric, F.Cu at (162.6, 70.7)
- added R118: 5k1, Resistor_SMD:R_0402_1005Metric, F.Cu at (165.5, 70.7)
- moved kibuzzard-665D4FC5 37.2 mm to (128.1, 68.3)
- moved kibuzzard-665D501B 30.2 mm to (148.5, 66.9)
- moved R116 4.40 mm to (174.1, 89.7)
- moved SW101 4.40 mm to (178.5, 88.3)
- moved SW102 4.40 mm to (178.5, 82.5)
- moved R106 4.39 mm to (174.1, 77.9)
- moved R115 4.39 mm to (174.1, 83.8)
- moved SW103 4.39 mm to (178.5, 76.6)
- moved kibuzzard-665D4EF8 4.39 mm to (170.0, 76.4)
- moved kibuzzard-665D4EFE 4.39 mm to (170.0, 82.4)
- moved kibuzzard-665D4F04 4.39 mm to (170.0, 88.1)
- moved C105 1.58 mm to (121.7, 101.0), turned to -90 degrees
- moved C106 1.10 mm to (126.6, 116.3)
- moved D103 0.76 mm to (120.0, 86.1)
- moved D104 0.76 mm to (120.0, 83.5)
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Connections:
- net Net-(CN10-Pin_1) renamed /C6
- net Net-(CN10-Pin_11) renamed /D4
- net Net-(CN10-Pin_12) renamed /R1
- net Net-(CN10-Pin_13) renamed /C3
- net Net-(CN10-Pin_14) renamed /R2
- net Net-(CN10-Pin_15) renamed /E4
- net Net-(CN10-Pin_16) renamed /T2
- net Net-(CN10-Pin_17) renamed /E3
- net Net-(CN10-Pin_18) renamed /R3
- net Net-(CN10-Pin_19) renamed /F4
- net Net-(CN10-Pin_2) renamed /M2
- net Net-(CN10-Pin_21) renamed /F3
- net Net-(CN10-Pin_22) renamed /R4
- net Net-(CN10-Pin_23) renamed /G4
- net Net-(CN10-Pin_24) renamed /T4
- net Net-(CN10-Pin_25) renamed /G3
- net Net-(CN10-Pin_26) renamed /R5
- net Net-(CN10-Pin_27) renamed /H3
- net Net-(CN10-Pin_28) renamed /R6
- net Net-(CN10-Pin_29) renamed /J4
- net Net-(CN10-Pin_3) renamed /D6
- net Net-(CN10-Pin_30) renamed /T6
- net Net-(CN10-Pin_31) renamed /J3
- net Net-(CN10-Pin_33) renamed /K4
- net Net-(CN10-Pin_34) renamed /R7
- net Net-(CN10-Pin_35) renamed /K3
- net Net-(CN10-Pin_37) renamed /R8
- net Net-(CN10-Pin_4) renamed /N1
- net Net-(CN10-Pin_5) renamed /C5
- net Net-(CN10-Pin_6) renamed /N3
- net Net-(CN10-Pin_8) renamed /P1
- net Net-(CN5-Pin_1) renamed /D11
- net Net-(CN5-Pin_10) renamed /F13
- net Net-(CN5-Pin_2) renamed /C11
- net Net-(CN5-Pin_3) renamed /D12
- net Net-(CN5-Pin_4) renamed /C12
- net Net-(CN5-Pin_5) renamed /D13
- net Net-(CN5-Pin_6) renamed /C13
- net Net-(CN5-Pin_9) renamed /E14
- net Net-(CN7-Pin_1) renamed /P14
- net Net-(CN7-Pin_13) renamed /K13
- net Net-(CN7-Pin_15) renamed /J14
- net Net-(CN7-Pin_17) renamed /J13
- net Net-(CN7-Pin_2) renamed /N13
- net Net-(CN7-Pin_21) renamed /H13
- net Net-(CN7-Pin_23) renamed /G14
- net Net-(CN7-Pin_25) renamed /G13
- net Net-(CN7-Pin_27) renamed /F14
- net Net-(CN7-Pin_28) renamed /A4
- net Net-(CN7-Pin_29) renamed /C1
- net Net-(CN7-Pin_3) renamed /M12
- net Net-(CN7-Pin_30) renamed /B4
- net Net-(CN7-Pin_31) renamed /C2
- net Net-(CN7-Pin_32) renamed /A3
- net Net-(CN7-Pin_33) renamed /D1
- net Net-(CN7-Pin_34) renamed /B3
- net Net-(CN7-Pin_35) renamed /D3
- net Net-(CN7-Pin_36) renamed /A2
- net Net-(CN7-Pin_37) renamed /B2
- net Net-(CN7-Pin_38) renamed /B1
- net Net-(CN7-Pin_4) renamed /P13
- net Net-(CN7-Pin_5) renamed /M13
- net Net-(CN7-Pin_7) renamed /L14
- net Net-(CN8-Pin_1) renamed /J2
- net Net-(CN8-Pin_2) renamed /K1
- net Net-(CN8-Pin_3) renamed /K2
- net Net-(CN8-Pin_4) renamed /L1
- net Net-(CN8-Pin_5) renamed /L2
- net Net-(CN8-Pin_6) renamed /M1
- net Net-(CN9-Pin_1) renamed /D7
- net Net-(CN9-Pin_2) renamed /C7
- net Net-(CN9-Pin_3) renamed /D8
- net Net-(CN9-Pin_4) renamed /C8
- net Net-(CN9-Pin_5) renamed /D9
- net Net-(CN9-Pin_6) renamed /C9
- net Net-(CN9-Pin_7) renamed /D10
- net Net-(CN9-Pin_8) renamed /C10
Routing:
- net GND: track 46.3 -> 65.6 mm, vias 53 -> 51
- net +5V: track 123.9 -> 141.3 mm
- net +3V3: track 199.4 -> 205.0 mm, vias 12 -> 14
- net Net-(J102B-H14): track 52.5 -> 48.1 mm
- net Net-(J102B-L13): track 62.7 -> 58.3 mm
- net Net-(J102B-K14): track 57.3 -> 52.9 mm
- net Net-(D110-K): track 0.00 -> 1.75 mm
- net Net-(D109-K): track 0.00 -> 1.74 mm
- net Net-(D102-K): track 36.0 -> 34.7 mm
- net Net-(D107-K): track 53.2 -> 52.5 mm
- net Net-(D105-K): track 46.4 -> 45.6 mm
- net Net-(D103-K): track 39.4 -> 38.6 mm
- net Net-(D104-K): track 42.8 -> 42.1 mm
- net Net-(D108-K): track 56.7 -> 55.9 mm
- net Net-(D106-K): track 49.8 -> 49.1 mm
