File: frosting.kicad_sch (KiCad schematic)
At the start: 45 parts, among them J101 HRO-Type-C-31-M-12, J102 iCESugar-Pro, SW101 USER3, SW102 USER2, SW103 USER1, U101 SRV05-4, U102 XC6206

Commit message: clean erc drc
Parts:
- added D109: 5VOK, LED_SMD:LED_0603_1608Metric, symbol Device:LED
- added D110: 3V3OK, LED_SMD:LED_0603_1608Metric, symbol Device:LED
- added H101, H102, H103: M3, MountingHole:MountingHole_3.2mm_M3_DIN965_Pad, symbol Mechanical:MountingHole_Pad
- added R117, R118: 5k1, Resistor_SMD:R_0402_1005Metric, symbol Device:R_Small_US
- D101, D102, D103, D104, D105, D106, D107, D108: LCSC ID 0603 -> C2290
Connections:
- net +3V3: now also D110.2 (A)
- net +5V: now also D109.2 (A)
- net GND: now also H101.1, H102.1, H103.1, R117.2, R118.2
- net C6: now reaches CN10.1 (Pin_1), J102.122 (C6)
- net D4: now reaches CN10.11 (Pin_11), J102.132 (D4)
- net R1: now reaches CN10.12 (Pin_12), J102.131 (R1)
- net C3: now reaches CN10.13 (Pin_13), J102.134 (C3)
- net R2: now reaches CN10.14 (Pin_14), J102.133 (R2)
- net E4: now reaches CN10.15 (Pin_15), J102.136 (E4)
- net T2: now reaches CN10.16 (Pin_16), J102.135 (T2)
- net E3: now reaches CN10.17 (Pin_17), J102.138 (E3)
- net R3: now reaches CN10.18 (Pin_18), J102.137 (R3)
- net F4: now reaches CN10.19 (Pin_19), J102.140 (F4)
- net M2: now reaches CN10.2 (Pin_2), J102.121 (M2)
- net F3: now reaches CN10.21 (Pin_21), J102.142 (F3)
- net R4: now reaches CN10.22 (Pin_22), J102.141 (R4)
- net G4: now reaches CN10.23 (Pin_23), J102.144 (G4)
- net T4: now reaches CN10.24 (Pin_24), J102.143 (T4)
- net G3: now reaches CN10.25 (Pin_25), J102.146 (G3)
- net R5: now reaches CN10.26 (Pin_26), J102.145 (R5)
- net H3: now reaches CN10.27 (Pin_27), J102.148 (H3)
- net R6: now reaches CN10.28 (Pin_28), J102.147 (R6)
- net J4: now reaches CN10.29 (Pin_29), J102.150 (J4)
- net D6: now reaches CN10.3 (Pin_3), J102.124 (D6)
- net T6: now reaches CN10.30 (Pin_30), J102.149 (T6)
- net J3: now reaches CN10.31 (Pin_31), J102.152 (J3)
- net K4: now reaches CN10.33 (Pin_33), J102.154 (K4)
- net R7: now reaches CN10.34 (Pin_34), J102.153 (R7)
- net K3: now reaches CN10.35 (Pin_35), J102.156 (K3)
- net R8: now reaches CN10.37 (Pin_37), J102.155 (R8)
- net N1: now reaches CN10.4 (Pin_4), J102.123 (N1)
- net C5: now reaches CN10.5 (Pin_5), J102.126 (C5)
- net N3: now reaches CN10.6 (Pin_6), J102.125 (N3)
- net P1: now reaches CN10.8 (Pin_8), J102.127 (P1)
- net D11: now reaches CN5.1 (Pin_1), J102.100 (D11)
- net F13: now reaches CN5.10 (Pin_10), J102.82 (F13)
- net C11: now reaches CN5.2 (Pin_2), J102.98 (C11)
- net D12: now reaches CN5.3 (Pin_3), J102.96 (D12)
- net C12: now reaches CN5.4 (Pin_4), J102.94 (C12)
- net D13: now reaches CN5.5 (Pin_5), J102.92 (D13)
- net C13: now reaches CN5.6 (Pin_6), J102.90 (C13)
- net E14: now reaches CN5.9 (Pin_9), J102.84 (E14)
- net J2: now reaches CN8.1 (Pin_1), J102.109 (J2)
- net K1: now reaches CN8.2 (Pin_2), J102.111 (K1)
- net K2: now reaches CN8.3 (Pin_3), J102.113 (K2)
- net L1: now reaches CN8.4 (Pin_4), J102.115 (L1)
- net L2: now reaches CN8.5 (Pin_5), J102.117 (L2)
- net M1: now reaches CN8.6 (Pin_6), J102.119 (M1)
- net C10: now reaches CN9.8 (Pin_8), J102.102 (C10)
- net D10: now reaches CN9.7 (Pin_7), J102.104 (D10)
- net C9: now reaches CN9.6 (Pin_6), J102.110 (C9)
- net D9: now reaches CN9.5 (Pin_5), J102.112 (D9)
- net C8: now reaches CN9.4 (Pin_4), J102.114 (C8)
- net D8: now reaches CN9.3 (Pin_3), J102.116 (D8)
- net C7: now reaches CN9.2 (Pin_2), J102.118 (C7)
- net D7: now reaches CN9.1 (Pin_1), J102.120 (D7)
- net C1: now reaches CN7.29 (Pin_29), J102.81 (C1)
- net C2: now reaches CN7.31 (Pin_31), J102.83 (C2)
- net D1: now reaches CN7.33 (Pin_33), J102.85 (D1)
- net D3: now reaches CN7.35 (Pin_35), J102.87 (D3)
- net P13: now reaches CN7.4 (Pin_4), J102.48 (P13)
- net N13: now reaches CN7.2 (Pin_2), J102.50 (N13)
- net P14: now reaches CN7.1 (Pin_1), J102.52 (P14)
- net M12: now reaches CN7.3 (Pin_3), J102.54 (M12)
- net M13: now reaches CN7.5 (Pin_5), J102.58 (M13)
- net L14: now reaches CN7.7 (Pin_7), J102.60 (L14)
- net K13: now reaches CN7.13 (Pin_13), J102.66 (K13)
- net A4: now reaches CN7.28 (Pin_28), J102.67 (A4)
- net J14: now reaches CN7.15 (Pin_15), J102.68 (J14)
- net B4: now reaches CN7.30 (Pin_30), J102.69 (B4)
- net J13: now reaches CN7.17 (Pin_17), J102.70 (J13)
- net A3: now reaches CN7.32 (Pin_32), J102.71 (A3)
- net B3: now reaches CN7.34 (Pin_34), J102.73 (B3)
- net H13: now reaches CN7.21 (Pin_21), J102.74 (H13)
- net A2: now reaches CN7.36 (Pin_36), J102.75 (A2)
- net G14: now reaches CN7.23 (Pin_23), J102.76 (G14)
- net B1: now reaches CN7.38 (Pin_38), J102.77 (B1)
- net G13: now reaches CN7.25 (Pin_25), J102.78 (G13)
- net B2: now reaches CN7.37 (Pin_37), J102.79 (B2)
- net F14: now reaches CN7.27 (Pin_27), J102.80 (F14)
- new net: D109.1 (K), R117.1
- new net: D110.1 (K), R118.1
- no-connect marks 26 -> 27
Other:
- moved on the sheet: C102, C103, C104, C105, C106, C107, C108, CN10, CN5, CN6, CN7, CN8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

Commit message: update grid origin and change 1x10P PN
Parts:
- CN5: LCSC ID C35445 -> C5116489
Changed lines of the file:
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@@
 			)
 		)
-		(property "LCSC ID" "C35445"
+		(property "LCSC ID" "C5116489"
 			(at 189.23 228.6 0)
 			(effects
